File: main_board/main_board.kicad_pcb (KiCad board)
At the start: 2 copper layers, 81 parts, among them J1 USB_C_Receptacle_USB2.0, J2 Conn_01x16, SW1 SW_Push, SW2 SW_Push, U1 W25Q128JVS, U10 AT42QT1011-TSHR, U11 AT42QT1011-TSHR, U12 AT42QT1011-TSHR, U13 AT42QT1011-TSHR, U14 AT42QT1011-TSHR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

Commit message: Main board complete?
Parts:
- removed C10, C11, C12, C13, C14, C6, C7, C8, C9: 100nF, Capacitor_SMD:C_0603_1608Metric_Pad1.08x0.95mm_HandSolder
- removed C15: 1uF, Capacitor_SMD:C_0603_1608Metric_Pad1.08x0.95mm_HandSolder
- removed C16, C17, C18, C22, C23, C24, C28, C29, C30, C34, C35, C36: 0.1uF, Capacitor_SMD:C_0603_1608Metric_Pad1.08x0.95mm_HandSolder
- removed C19, C20, C21, C25, C26, C27, C31, C32, C33, C37, C38, C39: 10nF, Capacitor_SMD:C_0603_1608Metric_Pad1.08x0.95mm_HandSolder
- removed C3: 27pF, Capacitor_SMD:C_0402_1005Metric_Pad0.74x0.62mm_HandSolder
- removed C4, C5: 10uF, Capacitor_SMD:C_0402_1005Metric_Pad0.74x0.62mm_HandSolder
- removed D1: LED_Small, LED_SMD:LED_0805_2012Metric_Pad1.15x1.40mm_HandSolder
- removed F1: Fuse_Small, Fuse:Fuse_1206_3216Metric_Pad1.42x1.75mm_HandSolder
- removed J2: Conn_01x16, Connector_FFC-FPC:TE_1-84952-6_1x16-1MP_P1.0mm_Horizontal
- removed R10, R11, R12, R13, R14, R15, R16, R17, R18, R19, R20, R9: 10k, Resistor_SMD:R_0603_1608Metric_Pad0.98x0.95mm_HandSolder
- removed R2: 5.1k, Resistor_SMD:R_0603_1608Metric_Pad0.98x0.95mm_HandSolder
- removed R3, R4: 27 Ohm, Resistor_SMD:R_0603_1608Metric_Pad0.98x0.95mm_HandSolder
- removed R5: DNF, Resistor_SMD:R_0402_1005Metric_Pad0.72x0.64mm_HandSolder
- removed R6, R7: 1k, Resistor_SMD:R_0402_1005Metric_Pad0.72x0.64mm_HandSolder
- removed R8: 10k, Resistor_SMD:R_0402_1005Metric_Pad0.72x0.64mm_HandSolder
- removed SW1, SW2: SW_Push, Button_Switch_THT:SW_PUSH_6mm
- removed U10, U11, U12, U13, U14, U15, U4, U5, U6, U7, U8, U9: AT42QT1011-TSHR, Package_TO_SOT_SMD:SOT-23-6
- removed U3: RP2040, RP2040_minimal:RP2040-QFN-56
- removed Y1: 12.000MHz, Crystal:Crystal_SMD_3225-4Pin_3.2x2.5mm_HandSoldering
- C1: value 100nF -> 0.1uF; footprint Capacitor_SMD:C_0402_1005Metric_Pad0.74x0.62mm_HandSolder -> Capacitor_SMD:C_0805_2012Metric_Pad1.18x1.45mm_HandSolder
- C2: value 27pF -> 0.1uF; footprint Capacitor_SMD:C_0402_1005Metric_Pad0.74x0.62mm_HandSolder -> Capacitor_SMD:C_0805_2012Metric_Pad1.18x1.45mm_HandSolder
- J1: value USB_C_Receptacle_USB2.0 -> Conn_01x16; footprint Connector_USB:USB_C_Receptacle_JAE_DX07S016JA1R1500 -> Connector_FFC-FPC:TE_1-84952-6_1x16-1MP_P1.0mm_Horizontal; moved to B.Cu
- R1: value 5.1k -> 75k; footprint Resistor_SMD:R_0603_1608Metric_Pad0.98x0.95mm_HandSolder -> Resistor_SMD:R_0805_2012Metric_Pad1.20x1.40mm_HandSolder
- U1: value W25Q128JVS -> Pico; footprint Package_SO:SOIC-8_5.23x5.23mm_P1.27mm -> MCU_RaspberryPi_and_Boards:RPi_Pico_SMD_TH
- U2: value NCP1117-3.3_SOT223 -> MPR121QR2; footprint Package_TO_SOT_SMD:SOT-223-3_TabPin2 -> Package_DFN_QFN:UQFN-20_3x3mm_P0.4mm
- moved U2 34.6 mm to (122.9, 75.8), turned to -135 degrees
- moved R1 23.3 mm to (120.4, 72.9), turned to 45 degrees
- moved J1 20.8 mm to (122.9, 85.8), turned to 180 degrees
- moved C2 15.3 mm to (122.5, 69.6), turned to -45 degrees
- moved U1 14.9 mm to (122.9, 64.3), turned to 0 degrees
- moved C1 9.69 mm to (125.8, 73.0), turned to -45 degrees
Connections:
- C1 pad 1: +3V3 -> GND
- C1 pad 2: GND -> +3V3
- C2 pad 2: XIN -> Net-(U2-VREG)
- R1 pad 1: Net-(J1-CC1) -> GND
- R1 pad 2: GND -> Net-(U2-REXT)
- U1 pad 1: QSPI_SS -> unconnected-(U1-GPIO0-Pad1)
- U1 pad 2: QSPI_SD1 -> unconnected-(U1-GPIO1-Pad2)
- U1 pad 3: QSPI_SD2 -> GND
- U1 pad 4: GND -> unconnected-(U1-GPIO2-Pad4)
- U1 pad 5: QSPI_SD0 -> unconnected-(U1-GPIO3-Pad5)
- U1 pad 6: QSPI_SCLK -> unconnected-(U1-GPIO4-Pad6)
- U1 pad 7: QSPI_SD3 -> unconnected-(U1-GPIO5-Pad7)
- U1 pad 8: +3V3 -> GND
- U2 pad 1: GND -> unconnected-(U2-~{IRQ}-Pad1)
- U2 pad 2: +3V3 -> SCL
- U2 pad 3: +5V -> SDA
Routing:
- net +3V3: track 84.5 -> 30.0 mm, vias 0 -> 1
- net RUN: track 42.0 -> 0.00 mm, vias 1 -> 0
- net Net-(R6-Pad1): track 26.9 -> 0.00 mm
- net QSPI_SD3: track 18.8 -> 0.00 mm
- net Net-(F1-Pad1): track 16.9 -> 0.00 mm, vias 2 -> 0
- net QSPI_SCLK: track 16.7 -> 0.00 mm
- net QSPI_SS: track 16.4 -> 0.00 mm
- net +1V1: track 14.5 -> 0.00 mm
- net QSPI_SD0: track 13.4 -> 0.00 mm
- net PAD0: track 0.00 -> 12.9 mm, vias 0 -> 1
- net PAD1: track 0.00 -> 11.7 mm, vias 0 -> 1
- net QSPI_SD1: track 11.3 -> 0.00 mm
- net USB D-: track 10.9 -> 0.00 mm
- net USB D+: track 10.8 -> 0.00 mm
- net QSPI_SD2: track 10.5 -> 0.00 mm
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- added copper zone on B.Cu, net GND
- added copper zone on F.Cu, net GND
Other:
- board outline added: 26 x 53 mm
- board text added: "LOW-KEY-AMUSE"
