File: main_board/main_board.kicad_pcb (KiCad board)
At the start: 2 copper layers, 26 x 53 mm, 10 parts, among them J1 Conn_01x16, U1 Pico, U2 MPR121QR2

Commit message: remove sneaky REF*** text
Other:
- board text added: "JLCJLCJLCJLC"
Changed lines of the file:
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@@
     (tags "mounting hole 2.1mm no annular")
     (attr exclude_from_pos_files exclude_from_bom)
-    (fp_text reference "REF**" (at 0 -3.2) (layer "F.SilkS")
+    (fp_text reference "REF**" (at 0 -3.2) (layer "F.SilkS") hide
         (effects (font (size 1 1) (thickness 0.15)))
     )
@@
   (gr_line (start 135 38) (end 111 38)
     (stroke (width 0.1) (type default)) (layer "Edge.Cuts"))
+  (gr_text "JLCJLCJLCJLC" (at 122.936 88.392) (layer "B.SilkS")
+    (effects (font (size 1 1) (thickness 0.15)) (justify bottom mirror))
+  )
   (gr_text "by dj505 & clue" (at 122.936 90.5764) (layer "F.SilkS")
     (effects (font (size 0.75 0.75) (thickness 0.15)) (justify bottom))

Commit message: Add code.py, update gerbers/prod files
Parts:
- removed REF** (x2): MountingHole_2.1mm, MountingHole:MountingHole_2.1mm
- added R2: 4.2k, Resistor_SMD:R_0805_2012Metric_Pad1.20x1.40mm_HandSolder, F.Cu at (124.5, 67.7)
- added R3: 4.2k, Resistor_SMD:R_0805_2012Metric_Pad1.20x1.40mm_HandSolder, F.Cu at (126.5, 65.6)
- C1, C2: value 0.1uF -> 100nF
Connections:
- J1 pad MP: GND -> (no net)
Routing:
- net +3V3: track 30.0 -> 50.1 mm
- net SCL: track 8.47 -> 17.3 mm
- net SDA: track 10.2 -> 15.7 mm
Other:
- board text added: "^ USB Port ^"
