File: keypad/keypad.kicad_sch (KiCad schematic)
At the start: 13 parts, among them J1 Conn_01x01, J10 Conn_01x01, J11 Conn_01x01, J12 Conn_01x01, J13 Conn_01x16, J2 Conn_01x01, J3 Conn_01x01, J4 Conn_01x01, J5 Conn_01x01, J6 Conn_01x01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

Commit message: Update keypad with ffc connector
Parts:
- J13: footprint Edge Connector:1.0mm Pitch Edge Connector 01x16 -> Connector_FFC-FPC:TE_1-84952-6_1x16-1MP_P1.0mm_Horizontal
Changed lines of the file:
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@@
       (effects (font (size 1.27 1.27)))
     )
-    (property "Footprint" "Edge Connector:1.0mm Pitch Edge Connector 01x16" (at 156.21 106.68 0)
+    (property "Footprint" "Connector_FFC-FPC:TE_1-84952-6_1x16-1MP_P1.0mm_Horizontal" (at 156.21 106.68 0)
       (effects (font (size 1.27 1.27)) hide)
     )
